Commit message: Added basic lidar

File: description/robot/robot.gazebo.xacro (robot description, xacro)
@@ -20,7 +20,9 @@
         <publish_link_pose>true</publish_link_pose>
         <use_pose_vector_msg>true</use_pose_vector_msg>
-        <!-- <publish_child_link_pose>true</publish_child_link_pose> New parameter -->
         <static_publisher>true</static_publisher>
         <static_update_frequency>1</static_update_frequency>
+      </plugin>
+      <plugin filename="gz-sim-sensors-system" name="gz::sim::systems::Sensors">
+        <render_engine>ogre2</render_engine>
       </plugin>
       <plugin
@@ -30,11 +32,4 @@
         <robot_base_frame>roboto</robot_base_frame>
       </plugin>
-        <plugin filename="gz-sim-diff-drive-system" name="gz::sim::systems::DiffDrive">
-    <left_joint>left_wheel_joint</left_joint>
-    <right_joint>right_wheel_joint</right_joint>
-    <wheel_separation>0.35</wheel_separation>
-    <wheel_radius>0.05</wheel_radius>
-    <max_acceleration>10.0</max_acceleration>
-  </plugin>
-        </gazebo>
+    </gazebo>
 </robot>

File: description/robot/robot_core.xacro (robot description, xacro)
@@ -115,4 +115,28 @@
         </xacro:inertial_sphere>
     </link>
+    <!-- LIDAR -->
+    <joint name="lidar_joint" type="fixed">
+        <parent link="base_link"/>
+        <child link="lidar_link"/>
+        <origin xyz="0.0 0.0 0.18"/>
+    </joint>
+   <link name="lidar_link">
+        <visual>
+            <geometry>
+                <box size="0.05 0.05 0.05"/>
+            </geometry>
+        </visual>
+        <collision>
+            <geometry>
+                <box size="0.05 0.05 0.05"/>
+            </geometry>
+        </collision>
+        <xacro:inertial_box mass="0.1" x="0.05" y="0.05" z="0.05">
+            <origin xyz="0 0 0" rpy="0 0 0"/>
+        </xacro:inertial_box>
+   </link>
+    <gazebo reference="lidar_joint">
+        <preserveFixedJoint>true</preserveFixedJoint>
+    </gazebo>
     <gazebo reference="chassis_joint">
         <preserveFixedJoint>true</preserveFixedJoint>
@@ -121,3 +145,34 @@
         <preserveFixedJoint>true</preserveFixedJoint>
     </gazebo>
+    <gazebo reference="lidar_link">
+        <sensor name='gpu_lidar' type='gpu_lidar'>"
+          <pose relative_to='lidar_link'>0 0 0 0 0 0</pose>
+          <topic>roboto/scan</topic>
+          <gz_frame_id>roboto/lidar_link</gz_frame_id>
+          <update_rate>5</update_rate>
+          <ray>
+              <scan>
+                  <horizontal>
+                      <samples>500</samples>
+                      <resolution>1</resolution>
+                      <min_angle>-3.14</min_angle>
+                      <max_angle>3.14</max_angle>
+                  </horizontal>
+                  <vertical>
+                      <samples>1</samples>
+                      <resolution>0.01</resolution>
+                      <min_angle>0</min_angle>
+                      <max_angle>0</max_angle>
+                  </vertical>
+              </scan>
+              <range>
+                  <min>0.08</min>
+                  <max>10.0</max>
+                  <resolution>0.01</resolution>
+              </range>
+          </ray>
+          <always_on>1</always_on>
+          <visualize>true</visualize>
+      </sensor>
+    </gazebo>
 </robot>
