Commit message: fixed bad odom, setup ready for nav2

File: description/robot/robot_core.xacro (robot description, xacro)
@@ -22,4 +22,11 @@
             <mass value="0.00001"/>
         </inertial> -->
+    </link>
+    <joint name="base_footprint_joint" type="fixed">
+        <parent link="base_link"/>
+        <child link="base_footprint"/>
+        <origin xyz="0.0 0.0 0.0" rpy="0.0 0.0 0.0"/>
+    </joint>
+    <link name="base_footprint">
     </link>
     <!-- CHASSIS LINK -->
@@ -57,5 +64,5 @@
         <visual>
             <geometry>
-                <cylinder radius="0.05" length="0.04"/>
+                    <sphere radius="0.05"/>
             </geometry>
             <material name="blue"/>
@@ -63,10 +70,10 @@
         <collision>
             <geometry>
-                <cylinder radius="0.05" length="0.04"/>
+                <sphere radius="0.05"/>
             </geometry>
         </collision>
-        <xacro:inertial_cylinder mass="0.1" length="0.04" radius="0.05">
+        <xacro:inertial_sphere mass="0.1" radius="0.05">
             <origin xyz="0 0 0" rpy="0 0 0"/>
-        </xacro:inertial_cylinder>
+        </xacro:inertial_sphere>
     </link>
     <!-- RIGHT WHEEL LINK -->
@@ -80,5 +87,5 @@
         <visual>
             <geometry>
-                <cylinder radius="0.05" length="0.04"/>
+                    <sphere radius="0.05"/>
             </geometry>
             <material name="blue"/>
@@ -86,10 +93,10 @@
         <collision>
             <geometry>
-                <cylinder radius="0.05" length="0.04"/>
+                <sphere radius="0.05"/>
             </geometry>
         </collision>
-        <xacro:inertial_cylinder mass="0.1" length="0.04" radius="0.05">
+        <xacro:inertial_sphere mass="0.1" radius="0.05">
             <origin xyz="0 0 0" rpy="0 0 0"/>
-        </xacro:inertial_cylinder>
+        </xacro:inertial_sphere>
     </link>
     <!-- CASTER WHEEL LINK -->

File: sim/gazebo/robot.gazebo.xacro (robot description, xacro)
@@ -71,7 +71,12 @@
     </vertical>
     </scan>
+    <noise>
+      <type>gaussian</type>
+      <mean>0.0</mean>
+      <stddev>0.007</stddev>
+    </noise>
     <range>
     <min>0.2</min>
-    <max>30.0</max>
+    <max>12.0</max>
     <resolution>0.01</resolution>
     </range>

Commit message: Added joystick control

File: description/robot/robot_core.xacro (robot description, xacro)
@@ -64,5 +64,5 @@
         <visual>
             <geometry>
-                    <sphere radius="0.05"/>
+                    <cylinder radius="0.05" length="0.04"/>
             </geometry>
             <material name="blue"/>
@@ -87,5 +87,6 @@
         <visual>
             <geometry>
-                    <sphere radius="0.05"/>
+                    <cylinder radius="0.05" length="0.04"/>
+                    <!-- <sphere radius="0.05"/> -->
             </geometry>
             <material name="blue"/>

Commit message: urdf corrections

File: description/robot/robot_core.xacro (robot description, xacro)
@@ -34,22 +34,22 @@
         <parent link="base_link"/>
         <child link="chassis"/>
-        <origin xyz="-0.1 0 0"/>
+        <origin xyz="-0.15 0 -0.0124"/>
     </joint>
     <link name="chassis">
         <visual>
-            <origin xyz="0.15 0 0.075"/>
+            <origin xyz="0.15 0 0.032"/>
             <geometry>
-                <box size="0.3 0.3 0.15"/>
+                <box size="0.3 0.15 0.064"/>
             </geometry>
             <material name="white"/>
         </visual>
         <collision>
-            <origin xyz="0.15 0 0.075"/>
+            <origin xyz="0.15 0 0.032"/>
             <geometry>
-                <box size="0.3 0.3 0.15"/>
+                <box size="0.3 0.15 0.064"/>
             </geometry>
         </collision>
-        <xacro:inertial_box mass="0.5" x="0.3" y="0.3" z="0.15">
-            <origin xyz="0.15 0 0.075" rpy="0 0 0"/>
+        <xacro:inertial_box mass="0.5" x="0.3" y="0.15" z="0.064">
+            <origin xyz="0.15 0 0.032" rpy="0 0 0"/>
         </xacro:inertial_box>
     </link>
@@ -58,5 +58,5 @@
         <parent link="base_link"/>
         <child link="left_wheel"/>
-        <origin xyz="0 0.175 0" rpy="-${pi/2} 0 0" />
+        <origin xyz="0 0.0822 0" rpy="-${pi/2} 0 0" />
         <axis xyz="0 0 1"/>
     </joint>
@@ -64,5 +64,5 @@
         <visual>
             <geometry>
-                    <cylinder radius="0.05" length="0.04"/>
+                    <cylinder radius="0.04" length="0.0128"/>
             </geometry>
             <material name="blue"/>
@@ -70,8 +70,8 @@
         <collision>
             <geometry>
-                <sphere radius="0.05"/>
+                <sphere radius="0.04"/>
             </geometry>
         </collision>
-        <xacro:inertial_sphere mass="0.1" radius="0.05">
+        <xacro:inertial_sphere mass="0.1" radius="0.04">
             <origin xyz="0 0 0" rpy="0 0 0"/>
         </xacro:inertial_sphere>
@@ -81,5 +81,5 @@
         <parent link="base_link"/>
         <child link="right_wheel"/>
-        <origin xyz="0 -0.175 0" rpy="${pi/2} 0 0" />
+        <origin xyz="0 -0.0822 0" rpy="${pi/2} 0 0" />
         <axis xyz="0 0 -1"/>
     </joint>
@@ -87,5 +87,5 @@
         <visual>
             <geometry>
-                    <cylinder radius="0.05" length="0.04"/>
+                    <cylinder radius="0.04" length="0.0128"/>
                     <!-- <sphere radius="0.05"/> -->
             </geometry>
@@ -94,8 +94,8 @@
         <collision>
             <geometry>
-                <sphere radius="0.05"/>
+                <sphere radius="0.04"/>
             </geometry>
         </collision>
-        <xacro:inertial_sphere mass="0.1" radius="0.05">
+        <xacro:inertial_sphere mass="0.1" radius="0.04">
             <origin xyz="0 0 0" rpy="0 0 0"/>
         </xacro:inertial_sphere>
@@ -103,12 +103,12 @@
     <!-- CASTER WHEEL LINK -->
     <joint name="caster_wheel_joint" type="fixed">
-        <parent link="chassis"/>
+        <parent link="base_link"/>
         <child link="caster_wheel"/>
-        <origin xyz="0.24 0 0"/>
+        <origin xyz="0.064 0 -0.025"/>
     </joint>
     <link name="caster_wheel">
         <visual>
             <geometry>
-                <sphere radius="0.05"/>
+                <sphere radius="0.015"/>
             </geometry>
             <material name="black"/>
@@ -116,8 +116,8 @@
         <collision>
             <geometry>
-                <sphere radius="0.05"/>
+                <sphere radius="0.015"/>
             </geometry>
         </collision>
-        <xacro:inertial_sphere mass="0.1" radius="0.05">
+        <xacro:inertial_sphere mass="0.1" radius="0.015">
             <origin xyz="0 0 0" rpy="0 0 0"/>
         </xacro:inertial_sphere>
@@ -127,18 +127,18 @@
         <parent link="base_link"/>
         <child link="lidar_link"/>
-        <origin xyz="0.0 0.0 0.18"/>
+        <origin xyz="0.1339 0.0 0.077"/>
     </joint>
    <link name="lidar_link">
         <visual>
             <geometry>
-                <box size="0.05 0.05 0.05"/>
+                <box size="0.0553 0.0553 0.044"/>
             </geometry>
         </visual>
         <collision>
             <geometry>
-                <box size="0.05 0.05 0.05"/>
+                <box size="0.0553 0.0553 0.044"/>
             </geometry>
         </collision>
-        <xacro:inertial_box mass="0.1" x="0.05" y="0.05" z="0.05">
+        <xacro:inertial_box mass="0.1" x="0.0553" y="0.0553" z="0.044">
             <origin xyz="0 0 0" rpy="0 0 0"/>
         </xacro:inertial_box>

Commit message: Basic working nav

File: description/robot/robot_core.xacro (robot description, xacro)
@@ -64,5 +64,5 @@
         <visual>
             <geometry>
-                    <cylinder radius="0.04" length="0.0128"/>
+                    <cylinder radius="0.0404" length="0.0128"/>
             </geometry>
             <material name="blue"/>
@@ -70,8 +70,8 @@
         <collision>
             <geometry>
-                <sphere radius="0.04"/>
+                <sphere radius="0.0404"/>
             </geometry>
         </collision>
-        <xacro:inertial_sphere mass="0.1" radius="0.04">
+        <xacro:inertial_sphere mass="0.1" radius="0.0404">
             <origin xyz="0 0 0" rpy="0 0 0"/>
         </xacro:inertial_sphere>
@@ -87,5 +87,5 @@
         <visual>
             <geometry>
-                    <cylinder radius="0.04" length="0.0128"/>
+                    <cylinder radius="0.0404" length="0.0128"/>
                     <!-- <sphere radius="0.05"/> -->
             </geometry>
@@ -94,8 +94,8 @@
         <collision>
             <geometry>
-                <sphere radius="0.04"/>
+                <sphere radius="0.0404"/>
             </geometry>
         </collision>
-        <xacro:inertial_sphere mass="0.1" radius="0.04">
+        <xacro:inertial_sphere mass="0.1" radius="0.0404">
             <origin xyz="0 0 0" rpy="0 0 0"/>
         </xacro:inertial_sphere>
@@ -127,5 +127,5 @@
         <parent link="base_link"/>
         <child link="lidar_link"/>
-        <origin xyz="0.1339 0.0 0.077"/>
+        <origin xyz="0.1339 0.0 0.077" rpy="0 0 ${pi}"/>
     </joint>
    <link name="lidar_link">

File: sim/gazebo/ros2_control.xacro (robot description, xacro)
@@ -12,5 +12,5 @@
         <param name="baud_rate">57600</param>
         <param name="timeout_ms">1000</param>
-        <param name="enc_counts_per_rev">1800</param>
+        <param name="enc_counts_per_rev">3587</param>
       </hardware>
       <joint name="left_wheel_joint">

Commit message: Added real robot urdf, launch cleanup

File: description/robot/robot_core.xacro (robot description, xacro)
@@ -2,24 +2,24 @@
 <robot xmlns:xacro="http://www.ros.org/wiki/xacro" >
     <xacro:include filename="inertial_macros.xacro"/>
-    <material name="white">
-        <color rgba="1 1 1 1" />
-    </material>
-    <material name="orange">
-        <color rgba="1 0.3 0.1 1"/>
-    </material>
-    <material name="blue">
-        <color rgba="0.2 0.2 1 1"/>
-    </material>
-    <material name="black">
-        <color rgba="0 0 0 1"/>
-    </material>
-    <!-- BASE LINK -->
+    <xacro:include filename="$(find roboto_diffbot)/description/robot/materials.xacro" />
     <link name="base_link">
-        <xacro:inertial_box mass="0.01" x="0.01" y="0.01" z="0.01">
-            <origin xyz="0 0 0" rpy="0 0 0"/>
-        </xacro:inertial_box>
-        <!-- <inertial>
-            <mass value="0.00001"/>
-        </inertial> -->
+    <inertial>
+        <origin xyz="-0.0022769860063732495 -0.0006106463755604264 0.0295548678674386" rpy="0 0 0"/>
+        <mass value="0.5933300696386302"/>
+        <inertia ixx="0.001482" iyy="0.002089" izz="0.002883" ixy="6.5e-05" iyz="1.2e-05" ixz="-0.0001"/>
+    </inertial>
+    <visual>
+        <origin xyz="0 0 0" rpy="0 0 0"/>
+        <geometry>
+        <mesh filename="file://$(find roboto_diffbot)/description/robot/meshes/base_link.stl" scale="0.001 0.001 0.001"/>
+        </geometry>
+        <material name="silver"/>
+    </visual>
+    <collision>
+        <origin xyz="0 0 0" rpy="0 0 0"/>
+        <geometry>
+        <mesh filename="file://$(find roboto_diffbot)/description/robot/meshes/base_link.stl" scale="0.001 0.001 0.001"/>
+        </geometry>
+    </collision>
     </link>
     <joint name="base_footprint_joint" type="fixed">
@@ -30,85 +30,90 @@
     <link name="base_footprint">
     </link>
-    <!-- CHASSIS LINK -->
-    <joint name="chassis_joint" type="fixed">
-        <parent link="base_link"/>
-        <child link="chassis"/>
-        <origin xyz="-0.15 0 -0.0124"/>
+    <link name="left_wheel">
+    <inertial>
+        <origin xyz="-4.928047540112002e-07 0.00649999998366961 1.4028976041274843e-07" rpy="0 0 0"/>
+        <mass value="0.06534512719466766"/>
+        <inertia ixx="2.7e-05" iyy="5.2e-05" izz="2.7e-05" ixy="0.0" iyz="0.0" ixz="0.0"/>
+    </inertial>
+    <visual>
+        <origin xyz="0.014004 -0.078 -0.021997" rpy="0 0 0"/>
+        <geometry>
+        <mesh filename="file://$(find roboto_diffbot)/description/robot/meshes/left_wheel_1.stl" scale="0.001 0.001 0.001"/>
+        </geometry>
+        <material name="silver"/>
+    </visual>
+    <collision>
+        <origin xyz="0.014004 -0.078 -0.021997" rpy="0 0 0"/>
+        <geometry>
+        <mesh filename="file://$(find roboto_diffbot)/description/robot/meshes/left_wheel_1.stl" scale="0.001 0.001 0.001"/>
+        </geometry>
+    </collision>
+    </link>
+    <link name="right_wheel">
+    <inertial>
+        <origin xyz="-4.928279983152511e-07 -0.006499999983669735 1.4028975616267592e-07" rpy="0 0 0"/>
+        <mass value="0.06534512719466772"/>
+        <inertia ixx="2.7e-05" iyy="5.2e-05" izz="2.7e-05" ixy="0.0" iyz="0.0" ixz="0.0"/>
+    </inertial>
+    <visual>
+        <origin xyz="0.014004 0.078 -0.021997" rpy="0 0 0"/>
+        <geometry>
+        <mesh filename="file://$(find roboto_diffbot)/description/robot/meshes/right_wheel_1.stl" scale="0.001 0.001 0.001"/>
+        </geometry>
+        <material name="silver"/>
+    </visual>
+    <collision>
+        <origin xyz="0.014004 0.078 -0.021997" rpy="0 0 0"/>
+        <geometry>
+        <mesh filename="file://$(find roboto_diffbot)/description/robot/meshes/right_wheel_1.stl" scale="0.001 0.001 0.001"/>
+        </geometry>
+    </collision>
+    </link>
+    <link name="lidar_link">
+    <inertial>
+        <origin xyz="1.0280064668785616e-05 1.1690792628638037e-07 0.012400389023013991" rpy="0 0 0"/>
+        <mass value="0.005290200757156612"/>
+        <inertia ixx="1e-06" iyy="1e-06" izz="2e-06" ixy="-0.0" iyz="-0.0" ixz="-0.0"/>
+    </inertial>
+    <visual>
+        <origin xyz="-0.067726 -0.0 -0.084534" rpy="0 0 0"/>
+        <geometry>
+        <mesh filename="file://$(find roboto_diffbot)/description/robot/meshes/lidar_link_1.stl" scale="0.001 0.001 0.001"/>
+        </geometry>
+        <material name="silver"/>
+    </visual>
+    <collision>
+        <origin xyz="-0.067726 -0.0 -0.084534" rpy="0 0 0"/>
+        <geometry>
+        <mesh filename="file://$(find roboto_diffbot)/description/robot/meshes/lidar_link_1.stl" scale="0.001 0.001 0.001"/>
+        </geometry>
+    </collision>
+    </link>
+    <joint name="left_wheel_joint" type="continuous">
+    <origin xyz="-0.014004 0.078 0.021997" rpy="0 0 0"/>
+    <parent link="base_link"/>
+    <child link="left_wheel"/>
+    <axis xyz="0.0 1.0 0.0"/>
     </joint>
-    <link name="chassis">
-        <visual>
-            <origin xyz="0.15 0 0.032"/>
-            <geometry>
-                <box size="0.3 0.15 0.064"/>
-            </geometry>
-            <material name="white"/>
-        </visual>
-        <collision>
-            <origin xyz="0.15 0 0.032"/>
-            <geometry>
-                <box size="0.3 0.15 0.064"/>
-            </geometry>
-        </collision>
-        <xacro:inertial_box mass="0.5" x="0.3" y="0.15" z="0.064">
-            <origin xyz="0.15 0 0.032" rpy="0 0 0"/>
-        </xacro:inertial_box>
-    </link>
-    <!-- LEFT WHEEL LINK -->
-    <joint name="left_wheel_joint" type="continuous">
-        <parent link="base_link"/>
-        <child link="left_wheel"/>
-        <origin xyz="0 0.0822 0" rpy="-${pi/2} 0 0" />
-        <axis xyz="0 0 1"/>
+    <joint name="right_wheel_joint" type="continuous">
+    <origin xyz="-0.014004 -0.078 0.021997" rpy="0 0 0"/>
+    <parent link="base_link"/>
+    <child link="right_wheel"/>
+    <axis xyz="-0.0 1.0 -0.0"/>
     </joint>
-    <link name="left_wheel">
-        <visual>
-            <geometry>
-                    <cylinder radius="0.0404" length="0.0128"/>
-            </geometry>
-            <material name="blue"/>
-        </visual>
-        <collision>
-            <geometry>
-                <sphere radius="0.0404"/>
-            </geometry>
-        </collision>
-        <xacro:inertial_sphere mass="0.1" radius="0.0404">
-            <origin xyz="0 0 0" rpy="0 0 0"/>
-        </xacro:inertial_sphere>
-    </link>
-    <!-- RIGHT WHEEL LINK -->
-    <joint name="right_wheel_joint" type="continuous">
-        <parent link="base_link"/>
-        <child link="right_wheel"/>
-        <origin xyz="0 -0.0822 0" rpy="${pi/2} 0 0" />
-        <axis xyz="0 0 -1"/>
+    <joint name="lidar_joint" type="fixed">
+    <origin xyz="0.067726 0.0 0.084534" rpy="0 0 0"/>
+    <parent link="base_link"/>
+    <child link="lidar_link"/>
     </joint>
-    <link name="right_wheel">
-        <visual>
-            <geometry>
-                    <cylinder radius="0.0404" length="0.0128"/>
-                    <!-- <sphere radius="0.05"/> -->
-            </geometry>
-            <material name="blue"/>
-        </visual>
-        <collision>
-            <geometry>
-                <sphere radius="0.0404"/>
-            </geometry>
-        </collision>
-        <xacro:inertial_sphere mass="0.1" radius="0.0404">
-            <origin xyz="0 0 0" rpy="0 0 0"/>
-        </xacro:inertial_sphere>
-    </link>
-    <!-- CASTER WHEEL LINK -->
     <joint name="caster_wheel_joint" type="fixed">
         <parent link="base_link"/>
         <child link="caster_wheel"/>
-        <origin xyz="0.064 0 -0.025"/>
+        <origin xyz="0.064 0 -0.012"/>
     </joint>
     <link name="caster_wheel">
         <visual>
             <geometry>
-                <sphere radius="0.015"/>
+                <sphere radius="0.0063"/>
             </geometry>
             <material name="black"/>
@@ -116,31 +121,10 @@
         <collision>
             <geometry>
-                <sphere radius="0.015"/>
+                <sphere radius="0.0063"/>
             </geometry>
         </collision>
-        <xacro:inertial_sphere mass="0.1" radius="0.015">
+        <xacro:inertial_sphere mass="0.02" radius="0.0063">
             <origin xyz="0 0 0" rpy="0 0 0"/>
         </xacro:inertial_sphere>
     </link>
-    <!-- LIDAR -->
-    <joint name="lidar_joint" type="fixed">
-        <parent link="base_link"/>
-        <child link="lidar_link"/>
-        <origin xyz="0.1339 0.0 0.077" rpy="0 0 ${pi}"/>
-    </joint>
-   <link name="lidar_link">
-        <visual>
-            <geometry>
-                <box size="0.0553 0.0553 0.044"/>
-            </geometry>
-        </visual>
-        <collision>
-            <geometry>
-                <box size="0.0553 0.0553 0.044"/>
-            </geometry>
-        </collision>
-        <xacro:inertial_box mass="0.1" x="0.0553" y="0.0553" z="0.044">
-            <origin xyz="0 0 0" rpy="0 0 0"/>
-        </xacro:inertial_box>
-   </link>
 </robot>

Commit message: new hardware integration

File: description/robot/robot_core.xacro (robot description, xacro)
@@ -103,5 +103,5 @@
     </joint>
     <joint name="lidar_joint" type="fixed">
-    <origin xyz="0.067726 0.0 0.084534" rpy="0 0 0"/>
+    <origin xyz="0.067726 0.0 0.084534" rpy="0 0 ${pi}"/>
     <parent link="base_link"/>
     <child link="lidar_link"/>

Commit message: small refactors

File: description/robot/robot_core.xacro (robot description, xacro)
@@ -59,5 +59,6 @@
         <origin xyz="0.014004 0.078 -0.021997" rpy="0 0 0"/>
         <geometry>
-        <mesh filename="file://$(find roboto_diffbot)/description/robot/meshes/right_wheel_1.stl" scale="0.001 0.001 0.001"/>
+        <mesh filename="file://$(find roboto_diffbot)/description/robot/meshes/right_wheel_1.stl"
+            scale="0.001 0.001 0.001"/>
         </geometry>
         <material name="silver"/>
@@ -66,8 +67,15 @@
         <origin xyz="0.014004 0.078 -0.021997" rpy="0 0 0"/>
         <geometry>
-        <mesh filename="file://$(find roboto_diffbot)/description/robot/meshes/right_wheel_1.stl" scale="0.001 0.001 0.001"/>
+        <mesh filename="file://$(find roboto_diffbot)/description/robot/meshes/right_wheel_1.stl"
+            scale="0.001 0.001 0.001"/>
         </geometry>
     </collision>
     </link>
+    <joint name="right_wheel_joint" type="continuous">
+        <origin xyz="-0.014004 -0.078 0.021997" rpy="0 0 0"/>
+        <parent link="base_link"/>
+        <child link="right_wheel"/>
+        <axis xyz="-0.0 1.0 -0.0"/>
+    </joint>
     <link name="lidar_link">
     <inertial>
@@ -95,10 +103,4 @@
     <child link="left_wheel"/>
     <axis xyz="0.0 1.0 0.0"/>
-    </joint>
-    <joint name="right_wheel_joint" type="continuous">
-    <origin xyz="-0.014004 -0.078 0.021997" rpy="0 0 0"/>
-    <parent link="base_link"/>
-    <child link="right_wheel"/>
-    <axis xyz="-0.0 1.0 -0.0"/>
     </joint>
     <joint name="lidar_joint" type="fixed">

File: sim/gazebo/ros2_control.xacro (robot description, xacro)
@@ -10,22 +10,13 @@
         <param name="loop_rate">30</param>
         <param name="can_interface">can0</param>
-        <!-- <param name="baud_rate">57600</param> -->
-        <!-- <param name="timeout_ms">1000</param> -->
-        <!-- <param name="enc_counts_per_rev">3587</param> -->
         <param name="enc_counts_per_rev">1793</param>
       </hardware>
       <joint name="left_wheel_joint">
-        <command_interface name="velocity">
-          <param name="min">-10</param>
-          <param name="max">10</param>
-        </command_interface>
+        <command_interface name="velocity"/>
         <state_interface name="position"/>
         <state_interface name="velocity"/>
       </joint>
       <joint name="right_wheel_joint">
-        <command_interface name="velocity">
-          <param name="min">-10</param>
-          <param name="max">10</param>
-        </command_interface>
+        <command_interface name="velocity"/>
         <state_interface name="position"/>
         <state_interface name="velocity"/>
@@ -39,16 +30,10 @@
       </hardware>
       <joint name="left_wheel_joint">
-        <command_interface name="velocity">
-          <param name="min">-10</param>
-          <param name="max">10</param>
-        </command_interface>
+        <command_interface name="velocity"/>
         <state_interface name="velocity"/>
         <state_interface name="position"/>
       </joint>
       <joint name="right_wheel_joint">
-        <command_interface name="velocity">
-          <param name="min">-10</param>
-          <param name="max">10</param>
-        </command_interface>
+        <command_interface name="velocity"/>
         <state_interface name="velocity"/>
         <state_interface name="position"/>
