Commit message: docking try 1

File: description/robot/robot_core.xacro (robot description, xacro)
@@ -98,4 +98,8 @@
     </collision>
     </link>
+    <link name="camera_link">
+    </link>
+    <link name="camera_link_optical">
+    </link>
     <joint name="left_wheel_joint" type="continuous">
     <origin xyz="-0.014004 0.078 0.021997" rpy="0 0 0"/>
@@ -108,4 +112,14 @@
     <parent link="base_link"/>
     <child link="lidar_link"/>
+    </joint>
+    <joint name="camera_joint" type="fixed">
+    <origin xyz="0.107726 0.0 0.064534" rpy="0 0 0"/>
+    <parent link="base_link"/>
+    <child link="camera_link"/>
+    </joint>
+    <joint name="camera_optical_joint" type="fixed">
+    <origin xyz="0 0 0" rpy="${-pi/2} 0 ${-pi/2}"/>
+    <parent link="camera_link"/>
+    <child link="camera_link_optical"/>
     </joint>
     <joint name="caster_wheel_joint" type="fixed">

File: sim/gazebo/robot.gazebo.xacro (robot description, xacro)
@@ -27,4 +27,26 @@
     <mu1 value="0.001"/>
     <mu2 value="0.001"/>
+  </gazebo>
+  <gazebo reference="camera_link">
+    <sensor name="camera" type="camera">
+      <pose> 0 0 0 0 0 0 </pose>
+      <visualize>true</visualize>
+      <update_rate>10</update_rate>
+      <camera>
+        <camera_info_topic>camera/camera_info</camera_info_topic>
+        <horizontal_fov>1.089</horizontal_fov>
+        <image>
+          <format>R8G8B8</format>
+          <width>640</width>
+          <height>480</height>
+        </image>
+        <clip>
+          <near>0.05</near>
+          <far>8.0</far>
+        </clip>
+      </camera>
+      <topic>camera/image_raw</topic>
+      <gz_frame_id>camera_link_optical</gz_frame_id>
+    </sensor>
   </gazebo>
   <gazebo reference="lidar_link">
