Commit message: basic real robot setup

File: sim/gazebo/ros2_control.gazebo.xacro (robot description, xacro)
@@ -2,5 +2,5 @@
 <robot xmlns:xacro="http://www.ros.org/wiki/xacro" >
     <!-- =============== Gazebo =============== -->
-  <ros2_control name="gazeboSystem" type="system">
+  <!-- <ros2_control name="gazeboSystem" type="system">
     <hardware>
       <plugin>gz_ros2_control/GazeboSimSystem</plugin>
@@ -22,4 +22,32 @@
       <state_interface name="position"/>
     </joint>
+  </ros2_control> -->
+  <ros2_control name="RealRobot" type="system">
+    <hardware>
+      <plugin>ros2_control_demo_example_2/DiffBotSystemHardware</plugin>
+      <param name="left_wheel_name">left_wheel_joint</param>
+      <param name="right_wheel_name">right_wheel_joint</param>
+      <param name="loop_rate">30</param>
+      <param name="device">/dev/ttyUSB0</param>
+      <param name="baud_rate">57600</param>
+      <param name="timeout_ms">1000</param>
+      <param name="enc_counts_per_rev">1800</param>
+    </hardware>
+    <joint name="left_wheel_joint">
+      <command_interface name="velocity">
+        <param name="min">-10</param>
+        <param name="max">10</param>
+      </command_interface>
+      <state_interface name="position"/>
+      <state_interface name="velocity"/>
+    </joint>
+    <joint name="right_wheel_joint">
+      <command_interface name="velocity">
+        <param name="min">-10</param>
+        <param name="max">10</param>
+      </command_interface>
+      <state_interface name="position"/>
+      <state_interface name="velocity"/>
+    </joint>
   </ros2_control>
 </robot>
